File: csi_project/LDO_hier.kicad_sch (KiCad schematic)
At the start: 8 parts, among them U1 LTC3035EDDBPBF

Commit message: Changed the value of a R and a few Cs
Parts:
- R6: value 210k -> 40k
Changed lines of the file:
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@@
 			)
 		)
-		(property "Value" "210k"
+		(property "Value" "40k"
 			(at 66.04 111.7599 0)
 			(effects
