File: csi_project/level_shifter_hier.kicad_sch (KiCad schematic)
At the start: 6 parts, among them U10 SN74LV1T34DBV, U11 SN74LV1T34DBV, U12 SN74LV1T34DBV, U13 SN74LV1T34DBV, U14 SN74LV1T34DBV, U15 SN74LV1T34DBV

Commit message: Fixed issues with Footprint assignment to main components,
Parts:
- U10, U11, U12, U13, U14, U15: footprint Package_TO_SOT_SMD:SOT-23-5 -> SN74LV1T34DBV:SN74LV1T34DBV
Changed lines of the file:
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@@
 			)
 		)
-		(property "Footprint" "Package_TO_SOT_SMD:SOT-23-5"
+		(property "Footprint" "SN74LV1T34DBV:SN74LV1T34DBV"
 			(at 166.37 114.3 0)
 			(effects
@@
 			)
 		)
-		(property "Footprint" "Package_TO_SOT_SMD:SOT-23-5"
+		(property "Footprint" "SN74LV1T34DBV:SN74LV1T34DBV"
 			(at 111.76 101.6 0)
 			(effects
@@
 			)
 		)
-		(property "Footprint" "Package_TO_SOT_SMD:SOT-23-5"
+		(property "Footprint" "SN74LV1T34DBV:SN74LV1T34DBV"
 			(at 179.07 139.7 0)
 			(effects
@@
 			)
 		)
-		(property "Footprint" "Package_TO_SOT_SMD:SOT-23-5"
+		(property "Footprint" "SN74LV1T34DBV:SN74LV1T34DBV"
 			(at 66.04 76.2 0)
 			(effects
@@
 			)
 		)
-		(property "Footprint" "Package_TO_SOT_SMD:SOT-23-5"
+		(property "Footprint" "SN74LV1T34DBV:SN74LV1T34DBV"
 			(at 88.9 88.9 0)
 			(effects
@@
 			)
 		)
-		(property "Footprint" "Package_TO_SOT_SMD:SOT-23-5"
+		(property "Footprint" "SN74LV1T34DBV:SN74LV1T34DBV"
 			(at 156.21 127 0)
 			(effects
